File: hardware/esp.seq/esp.seq.kicad_pcb (KiCad board)
At the start: 2 copper layers, 105.4 x 99.1 mm, 189 parts, among them J1 Conn_02x08, J10 PJ-301M-2, J11 PJ-301M-2, J12 PJ-301M-2, J13 PJ-301M-2, J14 PJ-301M-2, J15 PJ-301M-2, J16 PJ-301M-2, J17 PJ-301M-2, J18 PJ-301M-2, J19 PJ-301M-2, J2 USB-C, J20 PJ-301M-2, J21 PJ-301M-2, J22 PJ-301M-2, J23 Conn_01x04_Female, J24 Conn_01x04_Male, J25 Conn_01x06_Male, J26 Conn_01x06_Female, J3 USB-C, J4 Micro_SD_Card, J5 PJ-301M-3, J6 PJ-301M-3, J7 PJ-301M-2, J8 PJ-301M-2, J9 PJ-301M-2, U1 ESP32-S2-WROVER, U10 TL072, U11 TL072, U12 TL072, U2 AMS1117-3.3, U3 6N137, U4 CP2102, U5 TL072, U6 TL072, U7 TL072, U8 TL072, U9 TL072

Commit message: progress
Parts:
- removed D4: LED_Red, LED_THT:LED_D5.0mm
- removed R16: 220, Resistor_SMD:R_0805_2012Metric
- removed REF** (x2): MountingHole_3.2mm_M3, MountingHole:MountingHole_3.2mm_M3
- added C42: 1u, Capacitor_SMD:C_0805_2012Metric, F.Cu at (218.3, 100.2)
- added C43: 10u, Capacitor_SMD:C_0805_2012Metric, F.Cu at (231.2, 90.0)
- added C44: 100n, Capacitor_SMD:C_0805_2012Metric, F.Cu at (222.7, 96.5)
- added Q1: SS8050, Package_TO_SOT_SMD:SOT-323_SC-70, F.Cu at (218.3, 96.9)
- added Q2: SS8050, Package_TO_SOT_SMD:SOT-323_SC-70, F.Cu at (226.7, 90.3)
- added R101: 10k, Resistor_SMD:R_0402_1005Metric, F.Cu at (218.1, 107.6)
- added R102: 10k, Resistor_SMD:R_0402_1005Metric, F.Cu at (200.9, 117.8)
- added R103: 10k, Resistor_SMD:R_0402_1005Metric, F.Cu at (234.9, 89.5)
- C9: footprint Capacitor_SMD:C_1206_3216Metric -> Capacitor_SMD:C_0805_2012Metric
- J10, J11, J12, J13, J14, J15, J16, J17, J18, J19, J20, J21, J22, J7, J8, J9: footprint Connector_Audio:Jack_3.5mm_QingPu_WQP-PJ398SM_Vertical_CircularHoles -> lib:Jack_3.5mm_QingPu_WQP-PJ398SM_Vertical_CircularHoles
- J23: value Conn_01x04_Female -> Conn_01x04_Male; footprint Connector_PinSocket_2.54mm:PinSocket_1x04_P2.54mm_Vertical -> Connector_PinHeader_2.54mm:PinHeader_2x02_P2.54mm_Horizontal
- J24: footprint Connector_PinHeader_2.54mm:PinHeader_1x04_P2.54mm_Horizontal -> Connector_PinHeader_2.54mm:PinHeader_2x02_P2.54mm_Vertical; moved to B.Cu
- J25: footprint Connector_PinHeader_2.54mm:PinHeader_1x06_P2.54mm_Horizontal -> Connector_PinHeader_2.54mm:PinHeader_2x03_P2.54mm_Horizontal
- J26: value Conn_01x06_Female -> Conn_01x06_Male; footprint Connector_PinSocket_2.54mm:PinSocket_1x06_P2.54mm_Vertical -> Connector_PinHeader_2.54mm:PinHeader_2x03_P2.54mm_Vertical; moved to B.Cu
- R1, R10, R100, R11, R12, R13, R14, R15, R17, R18, R19, R2, R20, R21, R22, R23, R24, R25, R26, R27, R28, R29, R30, R31, R32, R33, R34, R35, R36, R37, R38, R39, R40, R41, R42, R43, R44, R45, R46, R47, R48, R49, R5, R50, R51, R52, R53, R54, R55, R56, R57, R58, R59, R6, R60, R61, R62, R63, R64, R65, R66, R67, R68, R69, R7, R70, R71, R72, R73, R74, R75, R76, R77, R78, R79, R8, R80, R81, R82, R83, R84, R85, R86, R87, R88, R89, R9, R90, R91, R92, R93, R94, R95, R96, R97, R98, R99: footprint Resistor_SMD:R_0805_2012Metric -> Resistor_SMD:R_0402_1005Metric
- R3, R4: footprint Resistor_SMD:R_0805_2012Metric -> Resistor_SMD:R_1206_3216Metric
- moved R1 310.0 mm to (110.5, 67.3)
- moved R61 293.7 mm to (192.3, 135.4)
- moved U9 283.3 mm to (186.4, 132.0)
- moved R99 281.3 mm to (247.3, 121.0)
- moved R79 280.7 mm to (189.4, 136.3)
- moved R64 279.7 mm to (202.3, 134.3)
- moved R69 278.8 mm to (201.0, 130.3)
- moved R65 278.0 mm to (196.5, 132.4)
- moved R76 277.3 mm to (183.6, 136.3)
- moved R96 277.2 mm to (241.5, 121.0)
- moved C26 277.2 mm to (197.3, 123.9)
- moved R91 275.2 mm to (258.9, 121.1)
- moved R2 275.1 mm to (110.5, 66.0)
- moved R81 274.5 mm to (250.2, 120.1)
- moved R71 274.0 mm to (201.1, 136.4)
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Connections:
- J23 pad 1: +5V -> Net-(D1-Pad1)
- J23 pad 2: USB_D- -> Net-(J23-Pad2)
- J23 pad 3: USB_D+ -> Net-(J23-Pad3)
- J23 pad 4: GND -> GND1
- J24 pad 1: Net-(D1-Pad1) -> +5V
- J24 pad 2: Net-(J24-Pad2) -> USB_D-
- J24 pad 3: Net-(J24-Pad3) -> USB_D+
- J24 pad 4: GND1 -> GND
- J3 pad A6: Net-(J24-Pad3) -> Net-(J23-Pad3)
- J3 pad A7: Net-(J24-Pad2) -> Net-(J23-Pad2)
- J3 pad B6: Net-(J24-Pad3) -> Net-(J23-Pad3)
- J3 pad B7: Net-(J24-Pad2) -> Net-(J23-Pad2)
- R100 pad 2: Out_43 -> OUT44
- R26 pad 1: IO3 -> IO2
- R30 pad 2: OUT13 -> OUT12
- R31 pad 1: IO2 -> IO3
- R35 pad 2: Out_11 -> OUT13
- R40 pad 2: Out_13 -> OUT14
- R45 pad 2: Out_21 -> OUT21
- R46 pad 1: IO7 -> IO6
- R50 pad 2: Out_23 -> OUT22
- R51 pad 1: IO6 -> IO7
- R55 pad 2: Out_21 -> OUT23
- R60 pad 2: Out_23 -> OUT24
- R65 pad 2: Out_31 -> OUT31
- R66 pad 1: IO11 -> IO10
- R70 pad 2: Out_33 -> OUT32
- R71 pad 1: IO10 -> IO11
- R75 pad 2: Out_31 -> OUT33
- R80 pad 2: Out_33 -> OUT34
- R85 pad 2: Out_41 -> OUT41
- R86 pad 1: IO15 -> IO14
- R90 pad 2: Out_43 -> OUT42
- R91 pad 1: IO14 -> IO15
- R95 pad 2: Out_41 -> OUT43
Other:
- board size 105.4 x 99.1 mm -> 58.4 x 119.4 mm

Commit message: footprint and layout updates
Parts:
- C8, D1, R1, R10, R2, R7, R8, R9: moved to B.Cu
- J10, J11, J12, J13, J14, J15, J16, J17, J18, J19, J20, J21, J22, J7, J8, J9: footprint lib:Jack_3.5mm_QingPu_WQP-PJ398SM_Vertical_CircularHoles -> lib:PJ-301M-2
- J2, J3: footprint Connector_USB:USB_C_Receptacle_HRO_TYPE-C-31-M-12 -> lib:TYPE-C-31-M-12; moved to B.Cu
- J4: footprint lib:SD-Card-DM3CS -> lib:HRS_DM3CS-SF; moved to B.Cu
- J5, J6: footprint lib:Jack_3.5mm_QingPu_WQP-PJ398SM_Vertical_CircularHoles-TRS -> lib:PJ-301M-3
- U1: footprint RF_Module:ESP32-S2-WROVER -> lib:ESP32-S2-WROVER; moved to F.Cu
- moved D1 110.5 mm to (108.0, 77.2)
- moved R10 86.1 mm to (143.3, 84.3), turned to 180 degrees
- moved R9 80.7 mm to (143.3, 81.3), turned to 180 degrees
- moved R8 74.7 mm to (143.3, 82.8)
- moved R7 71.5 mm to (143.3, 79.8), turned to 180 degrees
- moved C8 66.3 mm to (143.3, 87.1), turned to 180 degrees
- moved J2 52.4 mm to (152.4, 105.4), turned to -90 degrees
- moved J1 30.6 mm to (109.2, 115.6), turned to 0 degrees
- moved R1 19.0 mm to (119.9, 83.8), turned to -90 degrees
- moved R2 18.9 mm to (116.8, 83.8), turned to -90 degrees
- moved J3 9.59 mm to (118.1, 75.6), turned to 0 degrees
- moved J4 9.55 mm to (133.3, 80.7)
- moved J23 8.89 mm to (101.6, 74.9)
- moved J25 8.89 mm to (152.4, 74.9)
- moved U1 1.80 mm to (135.9, 105.4), turned to -90 degrees
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Connections:
- net Net-(C8-Pad1) renamed /CON_+3.3V
- net Net-(D1-Pad1) renamed /CON_+5V
- net Net-(D1-Pad2) renamed /CON_VBUS
- net Net-(J23-Pad2) renamed /CON_USB_D-
- net Net-(J23-Pad3) renamed /CON_USB_D+
- net Net-(J25-Pad2) renamed /CON_FSPI_CS
- net Net-(J25-Pad3) renamed /CON_FSPI_MOSI
- net Net-(J25-Pad4) renamed /CON_FSPI_CLK
- net Net-(J25-Pad5) renamed /CON_FSPI_MISO
- C8 pad 2: GND -> GND1
Routing:
- net GND1: track 0.00 -> 94.4 mm
- net /CON_FSPI_MISO: track 0.00 -> 47.7 mm
- net /CON_FSPI_CLK: track 0.00 -> 23.9 mm
- net /CON_FSPI_MOSI: track 0.00 -> 22.2 mm
- net /CON_+3.3V: track 0.00 -> 19.1 mm
- net /CON_FSPI_CS: track 0.00 -> 10.8 mm
- net /CON_+5V: track 0.00 -> 6.25 mm
Other:
- board size 58.4 x 119.4 mm -> 58.4 x 109.9 mm
