File: hardware/esp.seq/esp.seq.kicad_sch (KiCad schematic)
At the start: 67 parts, among them J1 Conn_02x08, J10 PJ-301M-2, J11 PJ-301M-2, J12 PJ-301M-2, J13 PJ-301M-2, J14 PJ-301M-2, J15 PJ-301M-2, J16 PJ-301M-2, J17 PJ-301M-2, J18 PJ-301M-2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

Commit message: progress
Parts:
- removed D3: 1N5819WS, Diode_SMD:D_SOD-323, symbol Diode:1N5819WS
- removed J23: Conn_01x04_Female, Connector_PinSocket_2.54mm:PinSocket_1x04_P2.54mm_Vertical, symbol Connector:Conn_01x04_Female
- removed J26: Conn_01x06_Female, Connector_PinSocket_2.54mm:PinSocket_1x06_P2.54mm_Vertical, symbol Connector:Conn_01x06_Female
- added C42: 1u, Capacitor_SMD:C_0805_2012Metric, symbol Device:C
- added C43: 10u, Capacitor_SMD:C_0805_2012Metric, symbol Device:C
- added C44: 100n, Capacitor_SMD:C_0805_2012Metric, symbol Device:C
- added D3: 1N5819WS, Diode_SMD:D_SOD-323, symbol Diode:1N5819
- added J24: Conn_01x04_Male, Connector_PinHeader_2.54mm:PinHeader_2x02_P2.54mm_Vertical, symbol Connector:Conn_01x04_Male
- added J26: Conn_01x06_Male, Connector_PinHeader_2.54mm:PinHeader_2x03_P2.54mm_Vertical, symbol Connector:Conn_01x06_Male
- added Q1, Q2: SS8050, Package_TO_SOT_SMD:SOT-323_SC-70, symbol Device:Q_NPN_BEC
- added R101, R102, R103: 10k, Resistor_SMD:R_0402_1005Metric, symbol Device:R
- C9: footprint Capacitor_SMD:C_1206_3216Metric -> Capacitor_SMD:C_0805_2012Metric; LCSC C1848 -> C28323
- D1: symbol Diode:1N5819WS -> Diode:1N5819
- D4: now left out of the parts list
- J10, J11, J12, J13, J14, J15, J16, J17, J18, J19, J20, J21, J22, J7, J8, J9: footprint Connector_Audio:Jack_3.5mm_QingPu_WQP-PJ398SM_Vertical_CircularHoles -> lib:Jack_3.5mm_QingPu_WQP-PJ398SM_Vertical_CircularHoles
- J23: renamed from J24; footprint Connector_PinHeader_2.54mm:PinHeader_1x04_P2.54mm_Horizontal -> Connector_PinHeader_2.54mm:PinHeader_2x02_P2.54mm_Horizontal
- J25: footprint Connector_PinHeader_2.54mm:PinHeader_1x06_P2.54mm_Horizontal -> Connector_PinHeader_2.54mm:PinHeader_2x03_P2.54mm_Horizontal
- R1, R11, R12, R2: footprint Resistor_SMD:R_0805_2012Metric -> Resistor_SMD:R_0402_1005Metric; LCSC C27834 -> C25905
- R10, R14, R7, R8, R9: footprint Resistor_SMD:R_0805_2012Metric -> Resistor_SMD:R_0402_1005Metric; LCSC C17713 -> C25792
- R13: footprint Resistor_SMD:R_0805_2012Metric -> Resistor_SMD:R_0402_1005Metric; LCSC C17560 -> C25768
- R15: footprint Resistor_SMD:R_0805_2012Metric -> Resistor_SMD:R_0402_1005Metric; LCSC C17513 -> C11702
- R16: footprint Resistor_SMD:R_0805_2012Metric -> Resistor_SMD:R_0402_1005Metric; LCSC C17557 -> C25091; now left out of the parts list
- R17, R18, R19, R20, R5: footprint Resistor_SMD:R_0805_2012Metric -> Resistor_SMD:R_0402_1005Metric; LCSC C17557 -> C25091
- R3, R4: footprint Resistor_SMD:R_0805_2012Metric -> Resistor_SMD:R_1206_3216Metric; LCSC C17714 -> C17936
- R6: footprint Resistor_SMD:R_0805_2012Metric -> Resistor_SMD:R_0402_1005Metric; LCSC C17710 -> C25117
- U3: symbol Isolator:6N137 -> lib:6N137
Connections:
- net +3.3V: now also C43.2, C44.2, J26.1 (Pin_1), R103.2
- net +5V: now also D3.1 (K), J24.1 (Pin_1)
- net DTR: now also Q2.2 (E), R101.1
- net EN: now also C42.1, Q1.3 (C), R103.1
- net FSPI_CLK: now also J26.4 (Pin_4)
- net FSPI_CS: now also J26.2 (Pin_2)
- net FSPI_MISO: now also J26.5 (Pin_5)
- net FSPI_MOSI: now also J26.3 (Pin_3)
- net GND: now also C42.2, C43.1, C44.1, J24.4 (Pin_4), J26.6 (Pin_6)
- net IO0: now also Q2.3 (C)
- net RTS: now also Q1.2 (E), R102.1
- net USB_D+: now also J24.3 (Pin_3)
- net USB_D-: now also J24.2 (Pin_2)
- net VBUS: now also D3.2 (A)
- new net: Q1.1 (B), R101.2
- new net: Q2.1 (B), R102.2
- no-connect marks 45 -> 49
Other:
- removed sheet Output-Stage-5
- removed sheet Output-Stage-6
- removed sheet Output-Stage-7
- removed sheet Output-Stage-8
- sheet Output-Stage-1 ports: added Out2 (5V), Out3 (10V), Out4 (10V), PWM3, PWM4; removed Out2 (10V)
- sheet Output-Stage-2 ports: added Out2 (5V), Out3 (10V), Out4 (10V), PWM3, PWM4; removed Out2 (10V)
- sheet Output-Stage-3 ports: added Out2 (5V), Out3 (10V), Out4 (10V), PWM3, PWM4; removed Out2 (10V)
- sheet Output-Stage-4 ports: added Out2 (5V), Out3 (10V), Out4 (10V), PWM3, PWM4; removed Out2 (10V)
- note added: "Power Flags"
- title: esp.seq -> esp.seq: Quad Output Stage
- moved on the sheet: C1, C2, C3, C4, C5, C6, C9, J1, R13, R14, R15, U1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

Commit message: footprint and layout updates
Parts:
- J10, J11, J12, J13, J14, J15, J16, J17, J18, J19, J20, J21, J22, J7, J8, J9: footprint lib:Jack_3.5mm_QingPu_WQP-PJ398SM_Vertical_CircularHoles -> lib:PJ-301M-2
- J2: footprint Connector_USB:USB_C_Receptacle_HRO_TYPE-C-31-M-12 -> lib:TYPE-C-31-M-12; LCSC C2927038 -> C165948
- J3: footprint Connector_USB:USB_C_Receptacle_HRO_TYPE-C-31-M-12 -> lib:TYPE-C-31-M-12; LCSC C2927038 -> C165948; Name USB Midi -> USB
- J4: footprint lib:SD-Card-DM3CS -> lib:HRS_DM3CS-SF; Name (none) -> Micro SD
- J5, J6: footprint lib:Jack_3.5mm_QingPu_WQP-PJ398SM_Vertical_CircularHoles-TRS -> lib:PJ-301M-3
- U1: footprint RF_Module:ESP32-S2-WROVER -> lib:ESP32-S2-WROVER
Connections:
- net GND: no longer C8.2
- net GND1: now also C8.2
- net CON_+3.3V: now reaches C8.1, J25.1 (Pin_1), J4.4 (VDD), R10.1, R7.1, R9.1
- net CON_FSPI_CS: now reaches J25.2 (Pin_2), J4.2 (DAT3/CD), R7.2
- net CON_FSPI_MOSI: now reaches J25.3 (Pin_3), J4.3 (CMD), R9.2
- net CON_FSPI_CLK: now reaches J25.4 (Pin_4), J4.5 (CLK), R8.1
- net CON_FSPI_MISO: now reaches J25.5 (Pin_5), J4.7 (DAT0), R10.2
- net CON_+5V: now reaches D1.1 (K), J23.1 (Pin_1)
- net CON_VBUS: now reaches D1.2 (A), J3.A4 (VBUS), J3.A9 (VBUS), J3.B4 (VBUS), J3.B9 (VBUS)
- net CON_USB_D+: now reaches J23.3 (Pin_3), J3.A6 (D+), J3.B6 (D+)
- net CON_USB_D-: now reaches J23.2 (Pin_2), J3.A7 (D-), J3.B7 (D-)
Other:
- moved on the sheet: D1
