File: hardware/esp.seq/output_stage.kicad_sch (KiCad schematic)
At the start: 15 parts, among them U5 TL072

Commit message: progress
Parts:
- added C14, C16: 470n, Capacitor_SMD:C_0805_2012Metric, symbol Device:C
- added C15, C17: 220n, Capacitor_SMD:C_0805_2012Metric, symbol Device:C
- added R31, R32, R36, R37: 10k, Resistor_SMD:R_0402_1005Metric, symbol Device:R
- added R33, R38: 220k, Resistor_SMD:R_0402_1005Metric, symbol Device:R
- added R34: 330k, Resistor_SMD:R_0402_1005Metric, symbol Device:R
- added R35, R40: 1k, Resistor_SMD:R_0402_1005Metric, symbol Device:R
- added R39: 100k, Resistor_SMD:R_0402_1005Metric, symbol Device:R
- added U6: TL072, Package_SO:SOIC-8_3.9x4.9mm_P1.27mm, symbol Amplifier_Operational:TL072
- R21, R22, R26, R27: footprint Resistor_SMD:R_0805_2012Metric -> Resistor_SMD:R_0402_1005Metric; LCSC C17414 -> C25744
- R23, R28: footprint Resistor_SMD:R_0805_2012Metric -> Resistor_SMD:R_0402_1005Metric; LCSC C17556 -> C25767
- R24: footprint Resistor_SMD:R_0805_2012Metric -> Resistor_SMD:R_0402_1005Metric; LCSC C17629 -> C25778
- R25, R30: footprint Resistor_SMD:R_0805_2012Metric -> Resistor_SMD:R_0402_1005Metric; LCSC C17513 -> C11702
- R29: footprint Resistor_SMD:R_0805_2012Metric -> Resistor_SMD:R_0402_1005Metric; LCSC C149504 -> C25741
Connections:
- net +12V: now also U6.8 (V+)
- net -12V: now also U6.4 (V-)
- net GND: now also C15.2, C17.2, R34.2, R39.2
- net Out2 (10V) renamed Out2 (5V)
- new net: C16.2, R36.2, R37.1
- new net: C17.1, R37.2, U6.5 (+)
- new net: C14.2, R31.2, R32.1
- new net: C16.1, R38.1, R40.1, U6.7
- new net: R33.2, R34.1, U6.2 (-)
- new net: C15.1, R32.2, U6.3 (+)
- new net: R38.2, R39.1, U6.6 (-)
- new net: C14.1, R33.1, R35.1, U6.1
- new net Out3 (10V): R35.2
- new net Out4 (10V): R40.2
- new net PWM3: R31.1
- new net PWM4: R36.1
Other:
- note added: "Non-inverting Amplifier"
- note added: "Output Stage 1, 2 (5V, Gain=1.67)"
- note added: "Output Stage 3, 4 (10V, Gain=3.2)"
- note removed: "Non-inverting Amplifier with Gain = 1.67"
- note removed: "Non-inverting Amplifier with Gain = 3.2"
- note removed: "Output Stage 1 (5V)"
- note removed: "Output Stage 2 (10V)"
- title: esp.seq: Dual Output Stage -> esp.seq: Quad Output Stage
- moved on the sheet: C10, C11, C12, C13, R21, R22, R23, R24, R25, R26, R27, R28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
